File: pcb/mainboard/ethernetPhy.sch (KiCad schematic (older format))
At the start: 0 parts

Commit message: worked on PoE regulator
Added the SRAM
Added an EEPROM and a FLASH as nonvolatileMemory
Parts:
- added C?: 1000p 2kV, symbol C
- added C?: 1u, symbol C
- added C?: 470p, symbol C
- added C?: 100n, symbol C
- added C?: 22n, symbol C
- added C?: 10n, symbol C
- added C?: 4.7u, symbol CP
- added D? (x2): D_Bridge_+-AA, symbol D_Bridge_+-AA
- added D?: SMAJ58A, symbol TVS_UNI
- added D?: BAS516, symbol D
- added L?: L, symbol L
- added R? (x4): 75, symbol R
- added R?: 0, symbol R
- added R? (x2): 270, symbol R
- added R?: 12k1, symbol R
- added R? (x3): 33, symbol R
- added R? (x4): 47k, symbol R
- added R?: 1k5, symbol R
- added R? (x4): 49.9, symbol R
- added R?: 68.1, symbol R
- added R? (x2): 10k, symbol R
- added R?: 6k8, symbol R
- added R?: 0.1, symbol R
- added TR?: H1102, symbol H1102
- added U?: LAN8720A, Housings_DFN_QFN:QFN-24-1EP_4x4mm_Pitch0.5mm, symbol LAN8720A
- added U?: USBLC6-4, symbol USBLC6-4
- added U?: ISM92-3251BH-50.0000, symbol OSC
- added U?: LTC4267, symbol LTC4267
Connections:
- new net: D?.1, D?.1 (+), D?.1 (+), R?.1, U?.13 (VPORTP)
- new net: D?.2, D?.2 (-), D?.2 (-), R?.1, U?.12 (SIGDISA), U?.7 (VPORTN)
- new net: D?.3, R?.1, TR?.15
- new net: D?.4, R?.1, TR?.10
- new net: R?.2, R?.2, U?.11 (CRS_DV/MODE2)
- new net: R?.1, U?.24 (RBIAS)
- new net: C?.1, C?.1, U?.6 (VDDCR)
- new net: R?.2, R?.2, U?.7 (RXD1/MODE1)
- new net: R?.2, R?.2, U?.8 (RXD0/MODE0)
- new net: C?.1, R?.2, R?.2, R?.2, R?.2
- new net: R?.2, U?.14 (SENSE)
- new net: D?.2 (A), U?.2 (ITH/RUN)
- new net: C?.1, R?.1, R?.2, U?.4 (PVCC)
- new net: R?.2, U?.5 (RCLASS)
- new net: R?.1, R?.2
- new net: D?.1 (K), R?.2
- new net +3V3_ETH: C?.1, L?.1, R?.1, R?.1, R?.1, R?.1, R?.1, U?.4 (VDD), U?.9 (VDDIO)
- new net CLK_OUT: U?.3 (OUT), U?.5 (XTAL1/CLKIN)
- new net CRS_DV: R?.1
- new net ETH1: TR?.16
- new net ETH2: TR?.14
- new net ETH3: TR?.11
- new net ETH4: D?.3, R?.1
- new net ETH6: TR?.9
- new net ETH7: D?.4, R?.1
- new net ETH_ACT_A: R?.2
- new net ETH_ACT_C: U?.2 (LED2/nINTSEL)
- new net ETH_LINK_A: U?.3 (LED1/REGOFF)
- new net ETH_LINK_C: R?.2
- new net ETH_SHIELD: C?.2, R?.1
- new net GND_ETH: C?.1, C?.2, C?.2, C?.2, C?.2, C?.2, R?.1, R?.1, R?.2, R?.2, U?.1 (PGND), U?.10 (POUT), U?.15 (VFB), U?.16 (PGND), U?.2 (GND), U?.2 (VSS), U?.25 (VSS), U?.8 (PGND), U?.9 (PGND)
- new net INT: R?.2, U?.14 (INT/REFCLKO)
- new net MDC: U?.13 (MDC)
- new net MDIO: R?.2, U?.12 (MDIO)
- new net RST: U?.15 (RST)
- new net RXD0: R?.1
- new net RXD1: R?.1
- new net RXER: U?.10 (RXER/PHYAD0)
- new net RX_N: R?.2, TR?.8, U?.22 (RXN), U?.3 (I/O2)
- new net RX_P: R?.2, TR?.6, U?.23 (RXP), U?.4 (I/O3)
- new net TXD0: U?.17 (TXD0)
- new net TXD1: U?.18 (TXD1)
- new net TXEN: U?.16 (TXEN)
- new net TX_N: R?.2, TR?.3, U?.20 (TXN), U?.6 (I/O4)
- new net TX_P: R?.2, TR?.1, U?.1 (I/O1), U?.21 (TXP)
- new net VDD_ETH: C?.1, C?.2, L?.2, R?.1, R?.1, R?.1, R?.1, R?.1, TR?.2, TR?.7, U?.1 (VDD2A), U?.19 (VDD1A), U?.5 (VBUS)
- no-connect marks 0 -> 2
