File: pcb/mainboard/nonvolatileMemory.sch (KiCad schematic (older format))
At the start: 0 parts

Commit message: worked on PoE regulator
Added the SRAM
Added an EEPROM and a FLASH as nonvolatileMemory
Parts:
- added U?: 24LC512, Housings_SOIC:SOIC-8_3.9x4.9mm_Pitch1.27mm, symbol 24LC512
- added U?: SST26VF064B, symbol SST26VF064B
Changed lines of the file:
@@
 $Descr A4 11693 8268
 encoding utf-8
-Sheet 1 10
-Title "ProzEthernatorMainboard"
+Sheet 6 10
+Title ""
 Date ""
-Rev "00"
-Comp "Shimatta"
+Rev ""
+Comp ""
 Comment1 ""
 Comment2 ""
@@
 Comment4 ""
 $EndDescr
+$Comp
+L 24LC512 U?
+U 1 1 5A86704E
+P 3300 2250
+F 0 "U?" H 3050 2500 50  0000 C CNN
+F 1 "24LC512" H 3350 2500 50  0000 L CNN
+F 2 "Housings_SOIC:SOIC-8_3.9x4.9mm_Pitch1.27mm" H 3350 2000 50  0001 L CNN
+F 3 "" H 3300 2150 50  0001 C CNN
+	1    3300 2250
+	1    0    0    -1
+$EndComp
+$Comp
+L SST26VF064B U?
+U 1 1 5A867804
+P 5050 4700
+F 0 "U?" H 5100 4550 60  0000 C CNN
+F 1 "SST26VF064B" H 5350 4650 60  0000 C CNN
+F 2 "" H 5050 4700 60  0001 C CNN
+F 3 "" H 5050 4700 60  0001 C CNN
+	1    5050 4700
+	1    0    0    -1
+$EndComp
 $EndSCHEMATC
